File: MSP430G2553IPW28_FT232RQ/MSP430G2553IPW28_FT232RQ.kicad_pcb (KiCad board)
At the start: 2 copper layers, 18.5 x 65.8 mm, 34 parts, among them IC1 MSP430G2553IPW28, IC2 FT232RQ, IC3 TLV74033PDBVR, J1 Conn_01x08_Male, J2 Conn_01x08_Male, J3 Conn_01x08_Male, J4 Conn_01x08_Male, P1 USB_C_Plug_USB2.0, SW1 SW_SPST, SW2 MSS22D18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

Commit message: update project
add 3d models and create new silkscreen elements.
Parts:
- moved G*** 3.05 mm to (134.9, 76.7)
- moved G*** 0.36 mm to (128.3, 84.3)
Other:
- board text added: "Apple Sauce"
- board text added: "DEC 2020"
- board text added: "Made in INDIA"
- board text removed: "DEC 2020 Apple Sauce"
