File: AppleSauce/AppleSauce.kicad_pcb (KiCad board)
At the start: 2 copper layers, 18.5 x 65.8 mm, 34 parts, among them IC1 MSP430G2553IPW28, IC2 FT232RQ, IC3 TLV74033PDBVR, J1 Conn_01x08_Male, J2 Conn_01x08_Male, J3 Conn_01x08_Male, J4 Conn_01x08_Male, P1 USB_C_Plug_USB2.0, SW1 SW_SPST, SW2 MSS22D18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

Commit message: Update Apple Sauce board
Other:
- board text added: "Designed in INDIA"
- board text removed: "Made in INDIA"
Changed lines of the file:
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@@
-(kicad_pcb (version 20171130) (host pcbnew 5.1.8-1.fc32)
+(kicad_pcb (version 20171130) (host pcbnew 5.1.9-1.fc32)
   (general
     (thickness 1.6)
@@
   )
   (page A4)
+  (title_block
+    (title "MSP430 Breadstick - Apple Sauce")
+    (date 2021-01-29)
+    (rev v0.1)
+    (company "Upside Down Labs")
+    (comment 2 "MSP430G2553IPW28 + FT232RQ")
+    (comment 3 "MSP430G2553 dev board")
+    (comment 4 "Upside Down Labs MSP430 Breadstick")
+  )
   (layers
     (0 F.Cu signal)
@@
     (effects (font (size 0.5 0.5) (thickness 0.125)) (justify mirror))
   )
-  (gr_text "Made in INDIA" (at 142.5 52.07 90) (layer B.SilkS)
-    (effects (font (size 1 1) (thickness 0.15)) (justify mirror))
+  (gr_text "Designed in INDIA" (at 142.9 52 90) (layer B.SilkS)
+    (effects (font (size 0.7 0.7) (thickness 0.15)) (justify mirror))
   )
   (gr_text "Apple Sauce" (at 129.54 52.078 90) (layer B.SilkS)
