File: CheeseDip/CheeseDip.kicad_pcb (KiCad board)
At the start: 2 copper layers, 21.6 x 60 mm, 92 parts, among them IC1 MSP430G2553IPW28, IC3 TLV74033PDBVR / ME6211, J1 Conn_02x06_Counter_Clockwise, J2 Conn_01x14, J5 Conn_01x14, P1 USB_C_Plug_USB2.0, SW1 SW_SPST, SW2 SS-3235S-L3, SW3 SW_SPST, U1 CH340C

Commit message: Update to v0.5
Parts:
- removed the ? at (151.3, 104.4)
- removed the ? at (151.1, 101.8)
- removed the ? at (150.8, 99.2)
- removed the ? at (151.1, 96.8)
- removed the ? at (151.1, 94.2)
- removed the ? at (151.1, 91.8)
- removed the ? at (151.1, 89.2)
- removed the ? at (150.8, 86.7)
- removed the ? at (150.8, 84.2)
- removed the ? at (150.8, 81.5)
- removed the ? at (137.9, 114.5)
- removed the ? at (137.9, 112.0)
- removed the ? at (137.9, 109.5)
- removed the ? at (137.9, 107.0)
- removed the ? at (137.9, 104.3)
- removed the ? at (137.9, 101.8)
- removed the ? at (137.9, 94.2)
- removed the ? at (137.9, 91.8)
- removed the ? at (137.9, 89.2)
- removed the ? at (137.9, 86.7)
- removed the ? at (137.9, 81.5)
- removed the ? at (137.9, 84.0)
- removed the ? at (137.9, 99.3)
- removed the ? at (137.9, 96.8)
- removed the ? at (151.1, 114.5)
- removed the ? at (151.1, 112.0)
- removed the ? at (151.8, 109.5)
- removed the ? at (151.1, 107.0)
- removed C5: 100nF, Capacitor_SMD:C_0603_1608Metric_Pad1.08x0.95mm_HandSolder
- removed P1: USB_C_Plug_USB2.0, Connector_USB:USB_C_Receptacle_HRO_TYPE-C-31-M-12
- added J3: USB_C_Receptacle_USB2.0, Connector_USB:USB_C_Receptacle_HRO_TYPE-C-31-M-12, F.Cu at (145.8, 60.6)
- moved R5 1.64 mm to (146.1, 91.3)
- moved C8 1.16 mm to (140.9, 103.0)
- moved ? 0.40 mm to (148.6, 81.5)
- moved ? 0.40 mm to (148.4, 89.3)
Connections:
- D1 pad 2: P1.5 -> P3.0
- SW1 pad 1: P1.2 -> P3.1
Routing:
- net P3.1: track 19.2 -> 42.4 mm, vias 1 -> 3
- net GND: track 164.0 -> 150.0 mm
- net P3.0: track 13.2 -> 19.7 mm
- net P1.2: track 40.5 -> 35.0 mm, vias 4 -> 2
- net D+: track 3.49 -> 7.63 mm, vias 0 -> 2
- net D-: track 3.81 -> 6.51 mm
- net DTR: track 66.8 -> 64.7 mm
- net P1.5: track 44.3 -> 42.6 mm
- net P1.1: track 44.0 -> 42.7 mm
- net P1.0: track 11.0 -> 10.1 mm
- net +3V3: track 88.2 -> 87.4 mm
- net P1.3: track 12.3 -> 12.9 mm
Other:
- board text added: "1"
- board text added: "10"
- board text added: "11"
- board text added: "12"
- board text added: "13"
- board text added: "14"
- board text added: "15"
- board text added: "16"
- board text added: "17"
- board text added: "18"
- board text added: "19"
- board text added: "2"
- board text added: "20"
- board text added: "21"
- board text added: "22"
- board text added: "23"
- board text added: "24"
- board text added: "3"
- board text added: "3V3"
- board text added: "4"
- board text added: "5"
- board text added: "5V"
- board text added: "6"
- board text added: "7"
- board text added: "8"
- board text added: "9"
- board text added: "FEB 2021 - v0.5"
- board text added: "P3.0"
- board text added: "P3.1"
- board text removed: "JAN 2020 - v0.2"
- board text removed: "P1.2"
- board text removed: "P1.5"
